File: CM4Emulator.kicad_sch (KiCad schematic)
At the start: 1 part, among them U1 Compute_Module_4_Functional

Commit message: audio and display changes
Other:
- moved on the sheet: U1B
Changed lines of the file:
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@@
 (kicad_sch (version 20230121) (generator eeschema)
   (paper "A4")
-  (symbol (lib_id "Raspberry_Pi_Compute_Module_4:Compute_Module_4_Functional") (at 115.57 60.96 0) (unit 2)
-    (in_bom yes) (on_board yes) (dnp no) (fields_autoplaced)
-    (property "Reference" "U1" (at 133.35 53.34 0)
+  (symbol (lib_id "Raspberry_Pi_Compute_Module_4:Compute_Module_4_Functional") (at 156.21 62.23 0) (mirror y) (unit 2)
+    (in_bom yes) (on_board yes) (dnp no)
+    (property "Reference" "U1" (at 138.43 54.61 0)
       (effects (font (size 1.524 1.524)))
     )
-    (property "Value" "Compute_Module_4_Functional" (at 133.35 55.88 0)
+    (property "Value" "Compute_Module_4_Functional" (at 138.43 57.15 0)
       (effects (font (size 1.524 1.524)))
     )
-    (property "Footprint" "RPi_Compute_Module_4:Raspberry-Pi-4-Compute-Module" (at 120.65 59.69 0)
+    (property "Footprint" "RPi_Compute_Module_4:Raspberry-Pi-4-Compute-Module" (at 151.13 60.96 0)
       (effects (font (size 1.524 1.524)) (justify left) hide)
     )
-    (property "Datasheet" "" (at 120.65 64.77 0)
+    (property "Datasheet" "" (at 151.13 66.04 0)
       (effects (font (size 1.524 1.524)) (justify left) hide)
     )
