File: HDMI.kicad_sch (KiCad schematic)
At the start: 2 parts, among them J1 HDMI_A, U2 Compute_Module_4_Functional

Commit message: added display things + others
Connections:
- net GND: now also J1.11 (CKS), J1.2 (D2S), J1.5 (D1S), J1.8 (D0S), J1.SH
- no-connect marks 0 -> 1
Changed lines of the file:
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@@
 (kicad_sch (version 20230121) (generator eeschema)
   (paper "A4")
+  (junction (at 197.485 129.54) (diameter 0) (color 0 0 0 0)
+  )
+  (junction (at 192.405 129.54) (diameter 0) (color 0 0 0 0)
+  )
+  (junction (at 200.025 129.54) (diameter 0) (color 0 0 0 0)
+  )
+  (junction (at 194.945 129.54) (diameter 0) (color 0 0 0 0)
+  )
+  (no_connect (at 184.785 113.03))
+  (wire (pts (xy 194.945 125.73) (xy 194.945 129.54))
+    (stroke (width 0) (type default))
+  )
   (wire (pts (xy 128.27 82.55) (xy 184.785 82.55))
     (stroke (width 0) (type default))
   )
   (wire (pts (xy 128.27 87.63) (xy 184.785 87.63))
+    (stroke (width 0) (type default))
+  )
+  (wire (pts (xy 192.405 129.54) (xy 194.945 129.54))
+    (stroke (width 0) (type default))
+  )
+  (wire (pts (xy 194.945 129.54) (xy 197.485 129.54))
     (stroke (width 0) (type default))
   )
@@
     (stroke (width 0) (type default))
   )
+  (wire (pts (xy 192.405 125.73) (xy 192.405 129.54))
+    (stroke (width 0) (type default))
+  )
   (wire (pts (xy 175.26 105.41) (xy 184.785 105.41))
     (stroke (width 0) (type default))
@@
     (stroke (width 0) (type default))
   )
+  (wire (pts (xy 202.565 125.73) (xy 202.565 129.54))
+    (stroke (width 0) (type default))
+  )
   (wire (pts (xy 128.27 110.49) (xy 136.525 110.49))
+    (stroke (width 0) (type default))
+  )
+  (wire (pts (xy 197.485 129.54) (xy 200.025 129.54))
     (stroke (width 0) (type default))
   )
@@
   )
   (wire (pts (xy 128.27 105.41) (xy 136.525 105.41))
+    (stroke (width 0) (type default))
+  )
+  (wire (pts (xy 200.025 129.54) (xy 200.025 130.81))
     (stroke (width 0) (type default))
   )
@@
     (stroke (width 0) (type default))
   )
-  (wire (pts (xy 200.025 125.73) (xy 200.025 130.81))
+  (wire (pts (xy 200.025 125.73) (xy 200.025 129.54))
     (stroke (width 0) (type default))
   )
@@
     (stroke (width 0) (type default))
   )
+  (wire (pts (xy 197.485 125.73) (xy 197.485 129.54))
+    (stroke (width 0) (type default))
+  )
+  (wire (pts (xy 202.565 129.54) (xy 200.025 129.54))
+    (stroke (width 0) (type default))
+  )
   (wire (pts (xy 128.27 102.87) (xy 136.525 102.87))
     (stroke (width 0) (type default))
   )
+  (wire (pts (xy 189.865 125.73) (xy 189.865 129.54))
+    (stroke (width 0) (type default))
+  )
+  (wire (pts (xy 189.865 129.54) (xy 192.405 129.54))
+    (stroke (width 0) (type default))
+  )

Commit message: audio and display changes
Connections:
- no-connect marks 1 -> 5
Changed lines of the file:
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@@
   (junction (at 194.945 129.54) (diameter 0) (color 0 0 0 0)
   )
+  (no_connect (at 80.01 102.87))
+  (no_connect (at 80.01 100.33))
   (no_connect (at 184.785 113.03))
+  (no_connect (at 80.01 105.41))
+  (no_connect (at 80.01 97.79))
   (wire (pts (xy 194.945 125.73) (xy 194.945 129.54))
     (stroke (width 0) (type default))
