File: CM4Emulator.kicad_pcb (KiCad board)
At the start: 2 copper layers, 4 parts, among them U1 Compute_Module_4_Functional, U2 TFP401APZP, U3 WM8960CGEFL/RV

Commit message: added display things + others
Parts:
- added U4: TUSB2046BVFR, easyeda2kicad:LQFP-32_L7.0-W7.0-P0.80-LS9.0-TL, F.Cu at (182.4, 74.5)
- moved FPC1 45.1 mm to (190.4, 115.2), turned to 180 degrees
- moved U2 0.80 mm to (188.5, 95.1)
Connections:
- FPC1 pad 1: unconnected-(FPC1-Pad1) -> /Display/LEDK
- FPC1 pad 10: unconnected-(FPC1-Pad10) -> /Display/R5
- FPC1 pad 11: unconnected-(FPC1-Pad11) -> /Display/R6
- FPC1 pad 12: unconnected-(FPC1-Pad12) -> /Display/R7
- FPC1 pad 13: unconnected-(FPC1-Pad13) -> /Display/G0
- FPC1 pad 14: unconnected-(FPC1-Pad14) -> /Display/G1
- FPC1 pad 15: unconnected-(FPC1-Pad15) -> /Display/G2
- FPC1 pad 16: unconnected-(FPC1-Pad16) -> /Display/G3
- FPC1 pad 17: unconnected-(FPC1-Pad17) -> /Display/G4
- FPC1 pad 18: unconnected-(FPC1-Pad18) -> /Display/G5
- FPC1 pad 19: unconnected-(FPC1-Pad19) -> /Display/G6
- FPC1 pad 2: unconnected-(FPC1-Pad2) -> +24V
- FPC1 pad 20: unconnected-(FPC1-Pad20) -> /Display/G7
- FPC1 pad 21: unconnected-(FPC1-Pad21) -> /Display/B0
- FPC1 pad 22: unconnected-(FPC1-Pad22) -> /Display/B1
- FPC1 pad 23: unconnected-(FPC1-Pad23) -> /Display/B2
- FPC1 pad 24: unconnected-(FPC1-Pad24) -> /Display/B3
- FPC1 pad 25: unconnected-(FPC1-Pad25) -> /Display/B4
- FPC1 pad 26: unconnected-(FPC1-Pad26) -> /Display/B5
- FPC1 pad 27: unconnected-(FPC1-Pad27) -> /Display/B6
- FPC1 pad 28: unconnected-(FPC1-Pad28) -> /Display/B7
- FPC1 pad 29: unconnected-(FPC1-Pad29) -> GND
- FPC1 pad 3: unconnected-(FPC1-Pad3) -> GND
- FPC1 pad 30: unconnected-(FPC1-Pad30) -> /Display/CLK
- FPC1 pad 31: unconnected-(FPC1-Pad31) -> /Display/ON/OFF
- FPC1 pad 32: unconnected-(FPC1-Pad32) -> /Display/HSYNC
- FPC1 pad 33: unconnected-(FPC1-Pad33) -> /Display/VSYNC
- FPC1 pad 34: unconnected-(FPC1-Pad34) -> /Display/DE
- FPC1 pad 36: unconnected-(FPC1-Pad36) -> GND
- FPC1 pad 4: unconnected-(FPC1-Pad4) -> VDD
- FPC1 pad 5: unconnected-(FPC1-Pad5) -> /Display/R0
- FPC1 pad 6: unconnected-(FPC1-Pad6) -> /Display/R1
- FPC1 pad 7: unconnected-(FPC1-Pad7) -> /Display/R2
- FPC1 pad 8: unconnected-(FPC1-Pad8) -> /Display/R3
- FPC1 pad 9: unconnected-(FPC1-Pad9) -> /Display/R4
- U1 pad 103: unconnected-(U1D-USB_N-Pad103) -> Net-(U1D-USB_N)
- U1 pad 105: unconnected-(U1D-USB_P-Pad105) -> Net-(U1D-USB_P)
- U2 pad 10: unconnected-(U2-QE0-Pad10) -> /Display/B0
- U2 pad 11: unconnected-(U2-QE1-Pad11) -> /Display/B1
- U2 pad 12: unconnected-(U2-QE2-Pad12) -> /Display/B2
- U2 pad 13: unconnected-(U2-QE3-Pad13) -> /Display/B3
- U2 pad 14: unconnected-(U2-QE4-Pad14) -> /Display/B4
- U2 pad 15: unconnected-(U2-QE5-Pad15) -> /Display/B5
- U2 pad 16: unconnected-(U2-QE6-Pad16) -> /Display/B6
- U2 pad 17: unconnected-(U2-QE7-Pad17) -> /Display/B7
- U2 pad 20: unconnected-(U2-QE8-Pad20) -> /Display/G0
- U2 pad 21: unconnected-(U2-QE9-Pad21) -> /Display/G1
- U2 pad 22: unconnected-(U2-QE10-Pad22) -> /Display/G2
- U2 pad 23: unconnected-(U2-QE11-Pad23) -> /Display/G3
- U2 pad 24: unconnected-(U2-QE12-Pad24) -> /Display/G4
- U2 pad 25: unconnected-(U2-QE13-Pad25) -> /Display/G5
- U2 pad 26: unconnected-(U2-QE14-Pad26) -> /Display/G6
- U2 pad 27: unconnected-(U2-QE15-Pad27) -> /Display/G7
- U2 pad 30: unconnected-(U2-QE16-Pad30) -> /Display/R0
- U2 pad 31: unconnected-(U2-QE17-Pad31) -> /Display/R1
- U2 pad 32: unconnected-(U2-QE18-Pad32) -> /Display/R2
- U2 pad 33: unconnected-(U2-QE19-Pad33) -> /Display/R3
- U2 pad 34: unconnected-(U2-QE20-Pad34) -> /Display/R4
- U2 pad 35: unconnected-(U2-QE21-Pad35) -> /Display/R5
- U2 pad 36: unconnected-(U2-QE22-Pad36) -> /Display/R6
- U2 pad 37: unconnected-(U2-QE23-Pad37) -> /Display/R7

Commit message: audio and display changes
Parts:
- added D1: SN75240PWR, easyeda2kicad:TSSOP-8_L4.4-W3.0-P0.65-LS6.4-BL, F.Cu at (219.6, 98.3)
- added J4: USB_C_Receptacle_USB2.0, Connector_USB:USB_C_Receptacle_HRO_TYPE-C-31-M-12, F.Cu at (216.0, 113.4)
Connections:
- U1 pad 84: unconnected-(U1A-CM4_3.3V_Out_1-Pad84) -> +3.3V
- U1 pad 86: unconnected-(U1A-CM4_3.3V_Out_2-Pad86) -> +3.3V
- U1 pad 88: unconnected-(U1A-CM4_1.8V_Out_1-Pad88) -> +1V8
- U1 pad 90: unconnected-(U1A-CM4_1.8V_Out_2-Pad90) -> +1V8
- U4 pad 25: unconnected-(U4-VCC-Pad25) -> +3.3V
- U4 pad 26: unconnected-(U4-~{EXTMEM}-Pad26) -> +3.3V
- U4 pad 27: unconnected-(U4-TSTPLL/48MCLK-Pad27) -> GND
- U4 pad 28: unconnected-(U4-GND-Pad28) -> GND
- U4 pad 29: unconnected-(U4-XTAL2-Pad29) -> Net-(U4-XTAL2)
- U4 pad 3: unconnected-(U4-VCC-Pad3) -> +3.3V
- U4 pad 30: unconnected-(U4-XTAL1-Pad30) -> Net-(U4-XTAL1)
- U4 pad 31: unconnected-(U4-TSTMODE-Pad31) -> GND
- U4 pad 6: unconnected-(U4-EEDATA/GANGED-Pad6) -> GND

Commit message: more display things
Parts:
- added RN1: YC164-JR-0710KL, easyeda2kicad:RES-ARRAY-SMD_0603-8P-L3.2-W1.6-BL, F.Cu at (214.3, 60.5)
- added RN2: YC164-JR-0710KL, easyeda2kicad:RES-ARRAY-SMD_0603-8P-L3.2-W1.6-BL, F.Cu at (217.4, 68.5)
- added RN3: YC164-JR-0710KL, easyeda2kicad:RES-ARRAY-SMD_0603-8P-L3.2-W1.6-BL, F.Cu at (217.4, 72.7)
- added RN4: YC164-JR-0710KL, easyeda2kicad:RES-ARRAY-SMD_0603-8P-L3.2-W1.6-BL, F.Cu at (217.4, 76.8)
- added RN5: YC164-JR-0710KL, easyeda2kicad:RES-ARRAY-SMD_0603-8P-L3.2-W1.6-BL, F.Cu at (217.4, 80.9)
- added RN6: YC164-JR-0710KL, easyeda2kicad:RES-ARRAY-SMD_0603-8P-L3.2-W1.6-BL, F.Cu at (217.4, 85.0)
- added RN7: YC164-JR-0710KL, easyeda2kicad:RES-ARRAY-SMD_0603-8P-L3.2-W1.6-BL, F.Cu at (217.4, 89.1)
Connections:
- FPC1 pad 10: /Display/R5 -> Net-(FPC1-Pad10)
- FPC1 pad 11: /Display/R6 -> Net-(FPC1-Pad11)
- FPC1 pad 12: /Display/R7 -> Net-(FPC1-Pad12)
- FPC1 pad 13: /Display/G0 -> Net-(FPC1-Pad13)
- FPC1 pad 14: /Display/G1 -> Net-(FPC1-Pad14)
- FPC1 pad 15: /Display/G2 -> Net-(FPC1-Pad15)
- FPC1 pad 16: /Display/G3 -> Net-(FPC1-Pad16)
- FPC1 pad 17: /Display/G4 -> Net-(FPC1-Pad17)
- FPC1 pad 18: /Display/G5 -> Net-(FPC1-Pad18)
- FPC1 pad 19: /Display/G6 -> Net-(FPC1-Pad19)
- FPC1 pad 20: /Display/G7 -> Net-(FPC1-Pad20)
- FPC1 pad 21: /Display/B0 -> Net-(FPC1-Pad21)
- FPC1 pad 22: /Display/B1 -> Net-(FPC1-Pad22)
- FPC1 pad 23: /Display/B2 -> Net-(FPC1-Pad23)
- FPC1 pad 24: /Display/B3 -> Net-(FPC1-Pad24)
- FPC1 pad 25: /Display/B4 -> Net-(FPC1-Pad25)
- FPC1 pad 26: /Display/B5 -> Net-(FPC1-Pad26)
- FPC1 pad 27: /Display/B6 -> Net-(FPC1-Pad27)
- FPC1 pad 28: /Display/B7 -> Net-(FPC1-Pad28)
- FPC1 pad 5: /Display/R0 -> Net-(FPC1-Pad5)
- FPC1 pad 6: /Display/R1 -> Net-(FPC1-Pad6)
- FPC1 pad 7: /Display/R2 -> Net-(FPC1-Pad7)
- FPC1 pad 8: /Display/R3 -> Net-(FPC1-Pad8)
- FPC1 pad 9: /Display/R4 -> Net-(FPC1-Pad9)
- U2 pad 18: unconnected-(U2-OVDD-Pad18) -> Net-(C25-Pad1)
- U2 pad 29: unconnected-(U2-OVDD-Pad29) -> Net-(C25-Pad1)
- U2 pad 38: unconnected-(U2-DVDD-Pad38) -> Net-(C22-Pad1)
- U2 pad 43: unconnected-(U2-OVDD-Pad43) -> Net-(C25-Pad1)
- U2 pad 44: unconnected-(U2-ODCK-Pad44) -> Net-(U2-ODCK)
- U2 pad 46: unconnected-(U2-DE-Pad46) -> Net-(U2-DE)
- U2 pad 47: unconnected-(U2-VSYNC-Pad47) -> Net-(U2-VSYNC)
- U2 pad 48: unconnected-(U2-HSYNC-Pad48) -> Net-(U2-HSYNC)
- U2 pad 57: unconnected-(U2-OVDD-Pad57) -> Net-(C25-Pad1)
- U2 pad 6: unconnected-(U2-DVDD-Pad6) -> Net-(C22-Pad1)
- U2 pad 67: unconnected-(U2-DVDD-Pad67) -> Net-(C22-Pad1)
- U2 pad 78: unconnected-(U2-OVDD-Pad78) -> Net-(C25-Pad1)
- U2 pad 82: unconnected-(U2-AVDD-Pad82) -> Net-(C30-Pad1)
- U2 pad 84: unconnected-(U2-AVDD-Pad84) -> Net-(C30-Pad1)
- U2 pad 88: unconnected-(U2-AVDD-Pad88) -> Net-(C30-Pad1)
- U2 pad 95: unconnected-(U2-AVDD-Pad95) -> Net-(C30-Pad1)
- U2 pad 97: unconnected-(U2-PVDD-Pad97) -> Net-(U2-PVDD)
- U3 pad 10: unconnected-(U3-DBVDD-Pad10) -> +3.3V
- U3 pad 19: unconnected-(U3-SPK_RN-Pad19) -> /Audio/SPK_RN
- U3 pad 20: unconnected-(U3-SPKGND2-Pad20) -> GND
- U3 pad 21: unconnected-(U3-SPKVDD2-Pad21) -> +3.3V
- U3 pad 22: unconnected-(U3-SPK_RP-Pad22) -> /Audio/SPK_RP
- U3 pad 23: unconnected-(U3-SPK_LN-Pad23) -> /Audio/SPK_LN
- U3 pad 24: unconnected-(U3-SPKGND1-Pad24) -> GND
- U3 pad 25: unconnected-(U3-SPK_LP-Pad25) -> /Audio/SPK_LP
- U3 pad 26: unconnected-(U3-SPKVDD1-Pad26) -> +3.3V
- U3 pad 28: unconnected-(U3-AGND-Pad28) -> GND
- U3 pad 29: unconnected-(U3-HP_R-Pad29) -> Net-(U3-HP_R)
- U3 pad 31: unconnected-(U3-HP_L-Pad31) -> Net-(U3-HP_L)
- U3 pad 32: unconnected-(U3-AVDD-Pad32) -> +3.3V
- U3 pad 8: unconnected-(U3-DCVDD-Pad8) -> +3.3V
- U3 pad 9: unconnected-(U3-DGND-Pad9) -> GND
