File: Display.kicad_sch (KiCad schematic)
At the start: 2 parts, among them U2 TFP401APZP

Commit message: added display things + others
Connections:
- net GND: now also FPC1.29, FPC1.3, FPC1.36
- net B0: now reaches U2.10 (QE0)
- net B0: now also FPC1.21
- net B1: now reaches U2.11 (QE1)
- net B1: now also FPC1.22
- net B2: now reaches U2.12 (QE2)
- net B2: now also FPC1.23
- net B3: now reaches U2.13 (QE3)
- net B3: now also FPC1.24
- net B4: now reaches U2.14 (QE4)
- net B4: now also FPC1.25
- net B5: now reaches U2.15 (QE5)
- net B5: now also FPC1.26
- net B6: now reaches U2.16 (QE6)
- net B6: now also FPC1.27
- net B7: now reaches U2.17 (QE7)
- net B7: now also FPC1.28
- net G0: now reaches U2.20 (QE8)
- net G0: now also FPC1.13
- net G1: now reaches U2.21 (QE9)
- net G1: now also FPC1.14
- net G2: now reaches U2.22 (QE10)
- net G2: now also FPC1.15
- net G3: now reaches U2.23 (QE11)
- net G3: now also FPC1.16
- net G4: now reaches U2.24 (QE12)
- net G4: now also FPC1.17
- net G5: now reaches U2.25 (QE13)
- net G5: now also FPC1.18
- net G6: now reaches U2.26 (QE14)
- net G6: now also FPC1.19
- net G7: now reaches U2.27 (QE15)
- net G7: now also FPC1.20
- net R0: now reaches U2.30 (QE16)
- net R0: now also FPC1.5
- net R1: now reaches U2.31 (QE17)
- net R1: now also FPC1.6
- net R2: now reaches U2.32 (QE18)
- net R2: now also FPC1.7
- net R3: now reaches U2.33 (QE19)
- net R3: now also FPC1.8
- net R4: now reaches U2.34 (QE20)
- net R4: now also FPC1.9
- net R5: now reaches U2.35 (QE21)
- net R5: now also FPC1.10
- net R6: now reaches U2.36 (QE22)
- net R6: now also FPC1.11
- net R7: now reaches U2.37 (QE23)
- net R7: now also FPC1.12
- net LEDK: now reaches FPC1.1
- net +24V: now reaches FPC1.2
- net CLK: now reaches FPC1.30
- net ON/OFF: now reaches FPC1.31
- net HSYNC: now reaches FPC1.32
- net VSYNC: now reaches FPC1.33
- net DE: now reaches FPC1.34
- net VDD: now reaches FPC1.4
- no-connect marks 0 -> 29
Other:
- note added: "No Touch (at least for now)"

Commit message: audio and display changes
Parts:
- added RN1, RN2, RN3, RN4, RN5, RN6, RN7: YC164-JR-0710KL, easyeda2kicad:RES-ARRAY-SMD_0603-8P-L3.2-W1.6-BL, symbol easyeda2kicad:YC164-JR-0710KL
Connections:
- net B0: now also RN5.5; no longer FPC1.21
- net B1: now also RN5.6; no longer FPC1.22
- net B2: now also RN5.7; no longer FPC1.23
- net B3: now also RN5.8; no longer FPC1.24
- net B4: now also RN6.5; no longer FPC1.25
- net B5: now also RN6.6; no longer FPC1.26
- net B6: now also RN6.7; no longer FPC1.27
- net B7: now also RN6.8; no longer FPC1.28
- net CLK: now also RN7.3
- net DE: now also RN7.4
- net G0: now also RN3.5; no longer FPC1.13
- net G1: now also RN3.6; no longer FPC1.14
- net G2: now also RN3.7; no longer FPC1.15
- net G3: now also RN3.8; no longer FPC1.16
- net G4: now also RN4.5; no longer FPC1.17
- net G5: now also RN4.6; no longer FPC1.18
- net G6: now also RN4.7; no longer FPC1.19
- net G7: now also RN4.8; no longer FPC1.20
- net HSYNC: now also RN7.1
- net R0: now also RN1.5; no longer FPC1.5
- net R1: now also RN1.6; no longer FPC1.6
- net R2: now also RN1.7; no longer FPC1.7
- net R3: now also RN1.8; no longer FPC1.8
- net R4: now also RN2.5; no longer FPC1.9
- net R5: now also RN2.6; no longer FPC1.10
- net R6: now also RN2.7; no longer FPC1.11
- net R7: now also RN2.8; no longer FPC1.12
- net VSYNC: now also RN7.2
- net at U2.44 (ODCK): now also RN7.6
- net at U2.46 (DE): now also RN7.5
- net at U2.47 (VSYNC): now also RN7.7
- net at U2.48 (HSYNC): now also RN7.8
- new net: FPC1.20, RN4.1
- new net: FPC1.19, RN4.2
- new net: FPC1.18, RN4.3
- new net: FPC1.17, RN4.4
- new net: FPC1.12, RN2.1
- new net: FPC1.11, RN2.2
- new net: FPC1.10, RN2.3
- new net: FPC1.9, RN2.4
- new net: FPC1.8, RN1.1
- new net: FPC1.7, RN1.2
- new net: FPC1.6, RN1.3
- new net: FPC1.5, RN1.4
- new net: FPC1.13, RN3.4
- new net: FPC1.14, RN3.3
- new net: FPC1.15, RN3.2
- new net: FPC1.16, RN3.1
- new net: FPC1.21, RN5.4
- new net: FPC1.22, RN5.3
- new net: FPC1.23, RN5.2
- new net: FPC1.24, RN5.1
- new net: FPC1.25, RN6.4
- new net: FPC1.26, RN6.3
- new net: FPC1.27, RN6.2
- new net: FPC1.28, RN6.1
- no-connect marks 29 -> 33
Other:
- moved on the sheet: FPC1, U2H

Commit message: more display things
Parts:
- added C17, C18, C19, C20, C23, C24, C26, C27, C28, C29, C31, C32, C33, C34: 0.1uF, symbol Device:C
- added C21, C22, C25, C30: 10uF, symbol Device:C
- added FB1, FB2, FB3, FB4: FerriteBead, symbol Device:FerriteBead
- added R5, R7: 10K, symbol Device:R
- added R6, R8: 0, symbol Device:R
Connections:
- net GND: now also U2.1 (DFO), U2.101 (EP), U2.4 (PIXS), C17.2, C18.2, C19.2, C20.2, C21.2, C22.2, C23.2, C24.2, C25.2, C26.2, C27.2, C28.2, C29.2, C30.2, C31.2, C32.2, C33.2, C34.2, R5.1, R8.1
- net at U2.100 (OCK_INV): now also R5.2, R6.2
- net at U2.18 (OVDD): now also U2.29 (OVDD), U2.43 (OVDD), U2.57 (OVDD), U2.78 (OVDD), C25.1, C26.1, C27.1, C28.1, C29.1, FB2.2
- net at U2.3 (ST): now also R7.2, R8.2
- net at U2.38 (DVDD): now also U2.6 (DVDD), U2.67 (DVDD), C22.1, C23.1, C24.1, FB3.2
- net +3.3V: now reaches U2.7 (~{STAG})
- net +3.3V: now also U2.99 (RSVD), FB1.1, FB2.1, FB3.1, FB4.1, R6.1, R7.1
- net at U2.82 (AVDD): now also U2.84 (AVDD), U2.88 (AVDD), U2.95 (AVDD), C30.1, C31.1, C32.1, C33.1, C34.1, FB1.2
- net at U2.97 (PVDD): now also C17.1, C18.1, C19.1, C20.1, C21.1, FB4.2
- no-connect marks 33 -> 36
Other:
- note added: "0Ohm resistors are used to change settings after manufacturing"
- note added: "still need to do LED power"
- moved on the sheet: U2H

Commit message: power changes
Connections:
- no-connect marks 36 -> 52
Changed lines of the file:
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@@
   (no_connect (at 209.55 111.76))
   (no_connect (at 308.61 172.72))
+  (no_connect (at 56.515 230.505))
   (no_connect (at 340.995 152.4))
+  (no_connect (at 56.515 258.445))
   (no_connect (at 209.55 88.9))
+  (no_connect (at 56.515 233.045))
   (no_connect (at 209.55 116.84))
   (no_connect (at 209.55 83.82))
@@
   (no_connect (at 209.55 86.36))
   (no_connect (at 209.55 214.63))
+  (no_connect (at 56.515 240.665))
   (no_connect (at 209.55 73.66))
   (no_connect (at 209.55 58.42))
@@
   (no_connect (at 209.55 78.74))
   (no_connect (at 209.55 219.71))
+  (no_connect (at 56.515 235.585))
+  (no_connect (at 56.515 225.425))
+  (no_connect (at 56.515 253.365))
   (no_connect (at 209.55 66.04))
+  (no_connect (at 56.515 238.125))
   (no_connect (at 308.61 170.18))
+  (no_connect (at 56.515 245.745))
   (no_connect (at 161.29 90.17))
   (no_connect (at 209.55 109.22))
   (no_connect (at 209.55 60.96))
+  (no_connect (at 56.515 248.285))
   (no_connect (at 209.55 106.68))
   (no_connect (at 308.61 165.1))
+  (no_connect (at 56.515 227.965))
+  (no_connect (at 56.515 260.985))
+  (no_connect (at 56.515 250.825))
   (no_connect (at 209.55 104.14))
   (no_connect (at 209.55 101.6))
+  (no_connect (at 56.515 255.905))
   (no_connect (at 209.55 55.88))
   (no_connect (at 209.55 63.5))
@@
   (no_connect (at 308.61 175.26))
   (no_connect (at 209.55 68.58))
+  (no_connect (at 56.515 222.885))
   (no_connect (at 161.29 58.42))
+  (no_connect (at 56.515 243.205))
   (no_connect (at 209.55 96.52))
   (no_connect (at 308.61 177.8))
