File: SD.kicad_sch (KiCad schematic)
At the start: 3 parts, among them J2 Micro_SD_Card, U2 Compute_Module_4_Functional

Commit message: power changes
Connections:
- no-connect marks 0 -> 6
Changed lines of the file:
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@@
   (junction (at 146.05 56.515) (diameter 0) (color 0 0 0 0)
   )
+  (no_connect (at 111.125 85.725))
+  (no_connect (at 111.125 88.265))
+  (no_connect (at 111.125 73.025))
+  (no_connect (at 111.125 83.185))
+  (no_connect (at 62.865 75.565))
+  (no_connect (at 111.125 78.105))
   (wire (pts (xy 148.59 71.755) (xy 142.875 71.755))
     (stroke (width 0) (type default))
