File: Unused.kicad_sch (KiCad schematic)
At the start: 1 part, among them U2 Compute_Module_4_Functional

Commit message: audio and display changes
Connections:
- no-connect marks 0 -> 28
Changed lines of the file:
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@@
 (kicad_sch (version 20230121) (generator eeschema)
   (paper "A4")
+  (no_connect (at 103.505 153.67))
+  (no_connect (at 103.505 146.05))
+  (no_connect (at 105.41 60.325))
+  (no_connect (at 103.505 158.75))
+  (no_connect (at 103.505 148.59))
+  (no_connect (at 103.505 130.81))
+  (no_connect (at 105.41 70.485))
+  (no_connect (at 46.99 60.325))
+  (no_connect (at 103.505 135.89))
+  (no_connect (at 105.41 52.705))
+  (no_connect (at 105.41 75.565))
+  (no_connect (at 103.505 151.13))
+  (no_connect (at 103.505 156.21))
+  (no_connect (at 103.505 163.83))
+  (no_connect (at 103.505 133.35))
+  (no_connect (at 105.41 62.865))
+  (no_connect (at 103.505 125.73))
+  (no_connect (at 103.505 143.51))
+  (no_connect (at 105.41 55.245))
+  (no_connect (at 105.41 57.785))
+  (no_connect (at 105.41 67.945))
+  (no_connect (at 103.505 128.27))
+  (no_connect (at 103.505 140.97))
+  (no_connect (at 105.41 73.025))
+  (no_connect (at 105.41 50.165))
+  (no_connect (at 103.505 161.29))
+  (no_connect (at 105.41 65.405))
+  (no_connect (at 103.505 138.43))
   (symbol (lib_id "Raspberry_Pi_Compute_Module_4:Compute_Module_4_Functional") (at 144.78 54.61 0) (unit 5)
     (in_bom yes) (on_board yes) (dnp no) (fields_autoplaced)

Commit message: power changes
Connections:
- no-connect marks 28 -> 37
Changed lines of the file:
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@@
 (kicad_sch (version 20230121) (generator eeschema)
   (paper "A4")
+  (no_connect (at 175.26 54.61))
   (no_connect (at 103.505 153.67))
   (no_connect (at 103.505 146.05))
@@
   (no_connect (at 105.41 75.565))
   (no_connect (at 103.505 151.13))
+  (no_connect (at 175.26 57.15))
+  (no_connect (at 175.26 59.69))
   (no_connect (at 103.505 156.21))
+  (no_connect (at 175.26 67.31))
   (no_connect (at 103.505 163.83))
   (no_connect (at 103.505 133.35))
   (no_connect (at 105.41 62.865))
+  (no_connect (at 175.26 62.23))
   (no_connect (at 103.505 125.73))
   (no_connect (at 103.505 143.51))
+  (no_connect (at 46.99 62.865))
   (no_connect (at 105.41 55.245))
+  (no_connect (at 175.26 72.39))
   (no_connect (at 105.41 57.785))
   (no_connect (at 105.41 67.945))
   (no_connect (at 103.505 128.27))
+  (no_connect (at 175.26 69.85))
+  (no_connect (at 175.26 64.77))
   (no_connect (at 103.505 140.97))
   (no_connect (at 105.41 73.025))
