File: _autosave-CM4Emulator.kicad_pcb (KiCad board)
At the start: 2 copper layers, 14 parts, among them J4 USB_C_Receptacle_USB2.0, U1 Compute_Module_4_Functional, U2 TFP401APZP, U3 WM8960CGEFL/RV, U4 TUSB2046BVFR

Commit message: power changes
Parts:
- added C35: 22uF, Capacitor_SMD:C_0805_2012Metric, F.Cu at (232.4, 73.6)
- added C36: 22uF, Capacitor_SMD:C_0805_2012Metric, F.Cu at (232.4, 76.7)
- added C37: 22uF, Capacitor_SMD:C_0805_2012Metric, F.Cu at (232.4, 79.7)
- added C38: 10nF, Capacitor_SMD:C_0402_1005Metric, F.Cu at (249.7, 83.8)
- added C39: 22uF, Capacitor_SMD:C_0805_2012Metric, F.Cu at (232.4, 82.7)
- added L1: 1uH, Inductor_SMD:L_0603_1608Metric, F.Cu at (228.2, 73.4)
- added R10: 100K, Resistor_SMD:R_0603_1608Metric, F.Cu at (228.2, 78.4)
- added R11: 1.0Meg, Resistor_SMD:R_0603_1608Metric, F.Cu at (228.2, 80.9)
- added R12: 5.6K, Resistor_SMD:R_0603_1608Metric, F.Cu at (228.2, 83.4)
- added R13: 0.2K, Resistor_SMD:R_0603_1608Metric, F.Cu at (228.2, 85.9)
- added R14: 10K, Resistor_SMD:R_0402_1005Metric, F.Cu at (246.8, 83.8)
- added R9: 402K, Resistor_SMD:R_0603_1608Metric, F.Cu at (228.2, 75.9)
- added SW1: SS-12D10L5, easyeda2kicad:SW-TH_SS-12D10L5, F.Cu at (239.6, 101.1)
- added U5: TPS61230DRCR, easyeda2kicad:VSON-10_L3.0-W3.0-P0.50-TL-EP_TPS61230DRCR, F.Cu at (242.9, 85.2)
- added U6: BQ24292IRGER, easyeda2kicad:QFN-24_L4.0-W4.0-P0.50-BL-EP2.7, F.Cu at (237.6, 85.7)
Connections:
- U1 pad 77: unconnected-(U1A-+5V-Pad77) -> +5V
- U1 pad 79: unconnected-(U1A-+5V-Pad79) -> +5V
- U1 pad 81: unconnected-(U1A-+5V-Pad81) -> +5V
- U1 pad 83: unconnected-(U1A-+5V-Pad83) -> +5V
- U1 pad 85: unconnected-(U1A-+5V-Pad85) -> +5V
- U1 pad 87: unconnected-(U1A-+5V-Pad87) -> +5V
- U2 pad 1: unconnected-(U2-DFO-Pad1) -> GND
- U2 pad 100: unconnected-(U2-OCK_INV-Pad100) -> Net-(U2-OCK_INV)
- U2 pad 101: unconnected-(U2-EP-Pad101) -> GND
- U2 pad 3: unconnected-(U2-ST-Pad3) -> Net-(U2-ST)
- U2 pad 4: unconnected-(U2-PIXS-Pad4) -> GND
- U2 pad 7: unconnected-(U2-~{STAG}-Pad7) -> +3.3V
- U2 pad 99: unconnected-(U2-RSVD-Pad99) -> +3.3V
